Commit message: 1440 mesh

File: config/urdf/combined.urdf (robot description, URDF)
Before this commit: robot combined, 19 links, 18 joints
Links:
- added link MA1440_base_link; collision mesh filename=model://MA_1440_A0/meshes/collision/base_link.stl; visual mesh filename=model://MA_1440_A0/meshes/visual/base_link.stl
- added link MA1440_link_1_s; collision mesh filename=model://MA_1440_A0/meshes/collision/link_1_s.stl; visual mesh filename=model://MA_1440_A0/meshes/visual/link_1_s.stl
- added link MA1440_link_2_l; collision mesh filename=model://MA_1440_A0/meshes/collision/link_2_l.stl; visual mesh filename=model://MA_1440_A0/meshes/visual/link_2_l.stl
- added link MA1440_link_3_u; collision mesh filename=model://MA_1440_A0/meshes/collision/link_3_u.stl; visual mesh filename=model://MA_1440_A0/meshes/visual/link_3_u.stl
- added link MA1440_link_4_r; collision mesh filename=model://MA_1440_A0/meshes/collision/link_4_r.stl; visual mesh filename=model://MA_1440_A0/meshes/visual/link_4_r.stl
- added link MA1440_link_5_b; collision mesh filename=model://MA_1440_A0/meshes/collision/link_5_b.stl; visual mesh filename=model://MA_1440_A0/meshes/visual/link_5_b.stl
- added link MA1440_link_6_t; collision mesh filename=model://MA_1440_A0/meshes/collision/link_6_t.stl; visual mesh filename=model://MA_1440_A0/meshes/visual/link_6_t.stl
- added link MA1440_tool0
Joints:
- added joint MA1440_joint_1_s: type revolute, parent MA1440_base_link, child MA1440_link_1_s, origin xyz=0 0 0.450 rpy=0 0 0, axis 0 0 1, limit lower=-2.9670 upper=2.9670 effort=648.27 velocity=3.8397
- added joint MA1440_joint_2_l: type revolute, parent MA1440_link_1_s, child MA1440_link_2_l, origin xyz=0.155 0 0 rpy=0 0 0, axis 0 1 0, limit lower=-1.5708 upper=2.7052 effort=874.65 velocity=3.4906
- added joint MA1440_joint_3_u: type revolute, parent MA1440_link_2_l, child MA1440_link_3_u, origin xyz=0 0 0.614 rpy=0 0 0, axis 0 -1 0, limit lower=-1.4835 upper=2.6179 effort=257.25 velocity=3.8397
- added joint MA1440_joint_4_r: type revolute, parent MA1440_link_3_u, child MA1440_link_4_r, origin xyz=0.640 0 0.200 rpy=0 0 0, axis -1 0 0, limit lower=-3.1415 upper=3.1415 effort=74.97 velocity=7.1558
- added joint MA1440_joint_5_b: type revolute, parent MA1440_link_4_r, child MA1440_link_5_b, origin xyz=0 0 0 rpy=0 0 0, axis 0 -1 0, limit lower=-2.3562 upper=2.3562 effort=44.69 velocity=7.1558
- added joint MA1440_joint_6_t: type revolute, parent MA1440_link_5_b, child MA1440_link_6_t, origin xyz=0 0 0 rpy=0 0 0, axis -1 0 0, limit lower=-6.2832 upper=6.2832 effort=14.80 velocity=10.6465
- added joint MA1440_joint_6_t-tool0: type fixed, parent MA1440_link_6_t, child MA1440_tool0, origin xyz=0.100 0 0 rpy=3.1415926 -1.570796 0
- added joint MA1440_pose: type fixed, parent world, child MA1440_base_link, origin xyz=4 0 0.0 rpy=0.0 0.0 3.14159

Commit message: urdf model finalize

File: config/urdf/combined.urdf (robot description, URDF)
Before this commit: robot combined, 27 links, 26 joints
Links:
- added link MA1440_pedestal; collision mesh filename=model://objects/meshes/ma1440_pedestal.stl scale=0.001 0.001 0.001; visual mesh filename=model://objects/meshes/ma1440_pedestal.stl scale=0.001 0.001 0.001
- added link MA2010_pedestal; collision box size=0.55 0.6858 0.762; visual box size=0.55 0.6858 0.762
Joints:
- added joint MA1440_joint_pedestal: type fixed, parent MA1440_base_link, child MA1440_pedestal, origin xyz=0 0 -0.908 rpy=0 0 0, axis 0 0 1
- added joint MA2010_joint_pedestal: type fixed, parent MA2010_base_link, child MA2010_pedestal, origin xyz=0 0 -0.381 rpy=0 0 0, axis 0 0 1
- joint D500B_pose: origin xyz=1.7482 -1.3208 0.0 rpy=0.0 0.0 1.57 -> xyz=1.7482 -1.3208 0.4688 rpy=0.0 0.260913569 1.57
- joint MA1440_joint_6_t-tool0: origin xyz=0.100 0 0 rpy=3.1415926 -1.570796 0 -> xyz=0 0 0 rpy=0 0 0
- joint MA1440_pose: origin xyz=4 0 0.0 rpy=0.0 0.0 3.14159 -> xyz=4 0 0.908 rpy=0.0 0.0 3.14159
- joint MA2010_pose: origin xyz=0.0 0 0.0 rpy=0.0 0.0 0.0 -> xyz=0.0 0 0.762 rpy=0.0 0.0 0.0

Commit message: invkin

File: config/urdf/combined.urdf (robot description, URDF)
Before this commit: robot combined, 29 links, 28 joints
Joints:
- joint D500B_pose: origin xyz=1.7482 -1.3208 0.4688 rpy=0.0 0.260913569 1.57 -> xyz=1.7482 -1.3208 0.4688 rpy=0.0 -0.260913569 -1.5708

Commit message: ready for welding

File: config/urdf/combined.urdf (robot description, URDF)
Before this commit: robot combined, 29 links, 28 joints
Links:
- added link weldgun; collision mesh filename=model://MA_2010_A0/meshes/collision/weldgun.stl scale=0.001 0.001 0.001; visual mesh filename=model://MA_2010_A0/meshes/visual/weldgun.stl scale=0.001 0.001 0.001
Joints:
- added joint weldgun_joint: type fixed, parent MA2010_link_6_t, child weldgun, origin xyz=0.1 0 0 rpy=0 1.57 0, axis 0 0 0
- joint D500B_pose: origin xyz=1.7482 -1.3208 0.4688 rpy=0.0 -0.260913569 -1.5708 -> xyz=1.645 -0.8446 0.4688 rpy=0.0 -0.261799 -1.5708

Commit message: octopuz calibration

File: config/urdf/combined.urdf (robot description, URDF)
Before this commit: robot combined, 30 links, 29 joints
Joints:
- joint D500B_pose: origin xyz=1.645 -0.8446 0.4688 rpy=0.0 -0.261799 -1.5708 -> xyz=1.6438 -0.911639 0.472054 rpy=0.0 -0.261799 -1.5708

Commit message: change urdf path

File: config/urdf/combined.urdf (robot description, URDF)
Before this commit: robot combined, 30 links, 29 joints
Links:
- link MA1440_tool0: geometry collision cylinder length=0.243 radius=0.05; visual cylinder length=0.243 radius=0.05
- link MA2010_base_link: geometry collision mesh filename=model://MA_2010_A0/meshes/collision/base_link.stl; visual mesh filename=../../config/urdf/MA_2010_A0/meshes/visual/base_link.stl
Joints:
- removed joint MA1440_joint_6_t-tool0
- added joint scanner_joint: type fixed, parent MA1440_link_6_t, child MA1440_tool0, origin xyz=-141.053 0 132.47 rpy=3.141592653589793 -1.2686793970944334 3.141592653589793, axis 0 0 0
- joint MA1440_pose: origin xyz=4 0 0.908 rpy=0.0 0.0 3.14159 -> xyz=2.7 -0.34 0.8 rpy=0.0 0.0 3.14159

Commit message: add scanner and holder urdf

File: config/urdf/combined.urdf (robot description, URDF)
Before this commit: robot combined, 30 links, 29 joints
Links:
- link Controller: geometry collision mesh filename=../../config/urdf/objects/meshes/controller.stl scale=0.001 0.001 0.001; visual mesh filename=../../config/urdf/objects/meshes/controller.stl scale=0.001 0.001 0.001
- link D500B_base_link: geometry collision mesh filename=../../config/urdf/D500B/meshes/collision/base_link.stl; visual mesh filename=../../config/urdf/D500B/meshes/visual/base_link.stl
- link D500B_link_1: geometry collision mesh filename=../../config/urdf/D500B/meshes/collision/link_1.stl; visual mesh filename=../../config/urdf/D500B/meshes/visual/link_1.stl
- link D500B_link_2: geometry collision mesh filename=../../config/urdf/D500B/meshes/collision/link_2.stl; visual mesh filename=../../config/urdf/D500B/meshes/visual/link_2.stl
- link MA1440_base_link: geometry collision mesh filename=../../config/urdf/MA_1440_A0/meshes/collision/base_link.stl; visual mesh filename=../../config/urdf/MA_1440_A0/meshes/visual/base_link.stl
- link MA1440_link_1_s: geometry collision mesh filename=../../config/urdf/MA_1440_A0/meshes/collision/link_1_s.stl; visual mesh filename=../../config/urdf/MA_1440_A0/meshes/visual/link_1_s.stl
- link MA1440_link_2_l: geometry collision mesh filename=../../config/urdf/MA_1440_A0/meshes/collision/link_2_l.stl; visual mesh filename=../../config/urdf/MA_1440_A0/meshes/visual/link_2_l.stl
- link MA1440_link_3_u: geometry collision mesh filename=../../config/urdf/MA_1440_A0/meshes/collision/link_3_u.stl; visual mesh filename=../../config/urdf/MA_1440_A0/meshes/visual/link_3_u.stl
- link MA1440_link_4_r: geometry collision mesh filename=../../config/urdf/MA_1440_A0/meshes/collision/link_4_r.stl; visual mesh filename=../../config/urdf/MA_1440_A0/meshes/visual/link_4_r.stl
- link MA1440_link_5_b: geometry collision mesh filename=../../config/urdf/MA_1440_A0/meshes/collision/link_5_b.stl; visual mesh filename=../../config/urdf/MA_1440_A0/meshes/visual/link_5_b.stl
- link MA1440_link_6_t: geometry collision mesh filename=../../config/urdf/MA_1440_A0/meshes/collision/link_6_t.stl; visual mesh filename=../../config/urdf/MA_1440_A0/meshes/visual/link_6_t.stl
- link MA1440_pedestal: geometry collision mesh filename=../../config/urdf/objects/meshes/ma1440_pedestal.stl scale=0.001 0.001 0.001; visual mesh filename=../../config/urdf/objects/meshes/ma1440_pedestal.stl scale=0.001 0.001 0.001
- link MA1440_tool0: geometry collision cylinder length=0.243 radius=0.05; visual cylinder length=0.243 radius=0.01
- link MA2010_base_link: geometry collision mesh filename=../../config/urdf/MA_2010_A0/meshes/collision/base_link.stl; visual mesh filename=../../config/urdf/MA_2010_A0/meshes/visual/base_link.stl
- link MA2010_link_1_s: geometry collision mesh filename=../../config/urdf/MA_2010_A0/meshes/collision/link_1_s.stl; visual mesh filename=../../config/urdf/MA_2010_A0/meshes/visual/link_1_s.stl
- link MA2010_link_2_l: geometry collision mesh filename=../../config/urdf/MA_2010_A0/meshes/collision/link_2_l.stl; visual mesh filename=../../config/urdf/MA_2010_A0/meshes/visual/link_2_l.stl
- link MA2010_link_3_u: geometry collision mesh filename=../../config/urdf/MA_2010_A0/meshes/collision/link_3_u.stl; visual mesh filename=../../config/urdf/MA_2010_A0/meshes/visual/link_3_u.stl
- link MA2010_link_4_r: geometry collision mesh filename=../../config/urdf/MA_2010_A0/meshes/collision/link_4_r.stl; visual mesh filename=../../config/urdf/MA_2010_A0/meshes/visual/link_4_r.stl
- link MA2010_link_5_b: geometry collision mesh filename=../../config/urdf/MA_2010_A0/meshes/collision/link_5_b.stl; visual mesh filename=../../config/urdf/MA_2010_A0/meshes/visual/link_5_b.stl
- link MA2010_link_6_t: geometry collision mesh filename=../../config/urdf/MA_2010_A0/meshes/collision/link_6_t.stl; visual mesh filename=../../config/urdf/MA_2010_A0/meshes/visual/link_6_t.stl
- link weldgun: geometry collision mesh filename=../../config/urdf/MA_2010_A0/meshes/collision/weldgun.stl scale=0.001 0.001 0.001; visual mesh filename=../../config/urdf/MA_2010_A0/meshes/visual/weldgun.stl scale=0.001 0.001 0.001
Joints:
- joint scanner_joint: origin xyz=-141.053 0 132.47 rpy=3.141592653589793 -1.2686793970944334 3.141592653589793 -> xyz=0.21347     0.    -0.222053 rpy=-0.30211692970046267  -0.0  -1.5707963267948966
