Commit message: urdf update

File: config/urdf/motoman_cell.urdf (robot description, URDF)
Before this commit: robot combined, 30 links, 29 joints
Links:
- added link Ground; collision box size=4.953 6.4 0.01; visual box size=4.953 6.4 0.01
- added link MA2010_filler; collision box size=0.3 0.5 0.3; visual box size=0.4 0.2 0.3
Joints:
- added joint Ground_pose: type fixed, parent world, child Ground, origin xyz=1.3462 0 -0.005 rpy=0.0 0.0 0
- added joint filler_joint: type fixed, parent MA2010_link_2_l, child MA2010_filler, origin xyz=0.0 -0.36 0.4 rpy=0 0 0, axis 0 0 0
- joint MA1440_pose: origin xyz=4 0 0.908 rpy=0.0 0.0 3.14159 -> xyz=2.689552 -0.39515 0.908 rpy=0.0 0.0 3.14159
